File: 04_schematics/Drone/droneV_0.1.kicad_sch (KiCad schematic)
At the start: 113 parts, among them J1 USB_C_Receptacle_USB2.0_14P, J2 Micro_SD_Card, J3 Conn_01x04_Pin, J4 Conn_01x05_Pin, J5 Conn_01x02_Pin, Q1 2N7002, SW1 SW_SPDT, SW2 SW_SPDT, U1 STM32F405RGT6, U2 LM2596S-5, U3 AMS1117-3.3, U4 MPU-6050, U5 HMC5883L, U6 SUP90P06-09L-E3, U7 nRF8001, Y1 16MHz, Y2 32.768 kHz, Y3 16MHz

Commit message: Screenshots of schematic and updated the schematic file
Parts:
- removed D10, D9: D_Schottky, symbol Device:D_Schottky
- removed D11, D12, D13, D14, D15, D4, D5, D6, D7, D8: D_TVS, symbol Device:D_TVS
- removed U6: SUP90P06-09L-E3, TO-220AB_VIS, symbol SUP90P06-09L:SUP90P06-09L-E3
- removed Y2: 32.768 kHz, Crystal:Crystal_SMD_3225-4Pin_3.2x2.5mm_HandSoldering, symbol Device:Crystal_GND24
- added C46: 1uF, symbol Device:C
- added D10, D11, D12, D13, D14, D4, D5, D7, D8, D9: SMBJ24CA_TR13, SMBJ24CA_TR13:DIONM5436X265N, symbol SMBJ24CA_TR13:SMBJ24CA_TR13
- added H1, H2, H3, H4: MountingHole, MountingHole:MountingHole_2.2mm_M2, symbol Mechanical:MountingHole
- added U6: SUP90P06-09L-E3, SUP90P06_09L_E3:TO-220AB_VIS, symbol SUP90P06_09L_E3:SUP90P06-09L-E3
- added U8: CH224K, Package_SO:SSOP-10-1EP_3.9x4.9mm_P1mm_EP2.1x3.3mm, symbol Interface_USB:CH224K
- added Y4: 16MHz, symbol Device:Crystal_GND24
- L1: value 33u -> 47u
- R7: value 5k1 -> 1k
- R8: value 5k1 -> 10k
- Y1: footprint Crystal:Crystal_SMD_3225-4Pin_3.2x2.5mm_HandSoldering -> (none); private (none) -> KLC_S4.1
- Y3: value 16MHz -> 32.768kHz; footprint Crystal:Crystal_SMD_3225-4Pin_3.2x2.5mm_HandSoldering -> (none); private (none) -> KLC_S4.1
Connections:
- net +3.3V: now also C4.1, D3.2 (A), R8.1, U3.2 (VO), D10.1, D12.1, D13.1, D14.1, D5.1, D7.1, D9.1
- net +5V: now also C2.1, D2.2 (A), L1.2, U2.4 (FB), D4.1; no longer J1.A4 (VBUS), J1.A9 (VBUS), J1.B4 (VBUS), J1.B9 (VBUS)
- net GND: now also C46.2, D10.2, D11.2, D12.2, D13.2, D14.2, D4.2, D5.2, D7.2, D8.2, D9.2, U8.11 (GND), U8.3 (CFG3), U8.9 (CFG1), Y4.2 (G), Y4.4 (G); no longer R7.1, R8.1
- net INT: now also U1.61 (PB8)
- net OSC_IN_16M: now also Y4.1; no longer Y3.1
- net OSC_IN_32k: now also Y3.1
- net OSC_OUT_16M: now also Y4.3; no longer Y3.3
- net OSC_OUT_32k: now also Y3.3
- net USB_D+: now also U8.4 (DP)
- net USB_D-: now also U8.5 (DM)
- net VBAT: now also D11.1, U6.2 (D)
- net VBAT_PRO: now also D8.1, U6.3 (S)
- net PG: now reaches U1.8 (PC0)
- net PG: now also R8.2, U8.10 (PG)
- net at Q1.3 (D), R15.2: now also U6.1 (G)
- net CC2: now reaches J1.B5 (CC2)
- net CC2: now also U8.6 (CC2); no longer R7.2
- net CC1: now reaches J1.A5 (CC1)
- net CC1: now also U8.7 (CC1); no longer R8.2
- net DRDY: no longer names the net of U5.5 (DRDY)
- net SCL_IMU renamed SCL
- net SDA_IMU renamed SDA
- new net VBUS: J1.A4 (VBUS), J1.A9 (VBUS), J1.B4 (VBUS), J1.B9 (VBUS), R7.1, U8.8 (VBUS)
- new net VDD: C46.1, R7.2, U8.1 (VDD), U8.2 (CFG2)
Other:
- note added: "MOUNTING HOLES"
- note added: "USB-C PROGRAMMING & CHARGER"
- note removed: "USB-C PROGRAMMING"
- company: (none) -> EYEFLY
- title: (none) -> EYEFLY V0.1
- moved on the sheet: C12, C33, C34, C35, C5, C6, C7, C8, C9, J1, R10, R3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

Commit message: nRF8001 DataSheet
Parts:
- removed AE1: Antenna, symbol Device:Antenna
- removed BZ1: Buzzer, symbol Device:Buzzer
- removed C1: 680u, symbol Device:C
- removed C10, C20, C25, C35, C7: 10u, symbol Device:C
- removed C11, C6, C8: 0.1u, symbol Device:C
- removed C12, C24: 4.7u, symbol Device:C
- removed C13, C16, C17, C18, C19, C21, C22, C26, C27, C29, C30, C31, C33, C34: 100n, symbol Device:C
- removed C14, C15: 10p, symbol Device:C
- removed C2: 220u, symbol Device:C
- removed C23, C32: 1u, symbol Device:C
- removed C28: 33n, symbol Device:C
- removed C3, C4: 22u, symbol Device:C
- removed C36, C37, C38, C39: 9p, symbol Device:C
- removed C40: 1.8p, symbol Device:C
- removed C41: N/C, symbol Device:C
- removed C42, C9: 2.2n, symbol Device:C
- removed C43: 1.2p, symbol Device:C
- removed C44, C45: 2.2u, symbol Device:C
- removed C46: 1uF, symbol Device:C
- removed C5: 10n, symbol Device:C
- removed D1: 1N5822, Diode_THT:D_DO-201AD_P15.24mm_Horizontal, symbol Diode:1N5822
- removed D10, D11, D12, D13, D14, D4, D5, D7, D8, D9: SMBJ24CA_TR13, SMBJ24CA_TR13:DIONM5436X265N, symbol SMBJ24CA_TR13:SMBJ24CA_TR13
- removed D16, D3: GREEN, symbol Device:LED
- removed D2: YELLOW, symbol Device:LED
- removed FB1, FB2: 120R, symbol Device:FerriteBead
- removed J1: USB_C_Receptacle_USB2.0_14P, symbol Connector:USB_C_Receptacle_USB2.0_14P
- removed J2: Micro_SD_Card, symbol Connector:Micro_SD_Card
- removed J3: Conn_01x04_Pin, symbol Connector:Conn_01x04_Pin
- removed J4: Conn_01x05_Pin, symbol Connector:Conn_01x05_Pin
- removed J5: Conn_01x02_Pin, symbol Connector:Conn_01x02_Pin
- removed L1: 47u, symbol Device:L
- removed L2: 8.2n, symbol Device:L
- removed L3: 3.9n, symbol Device:L
- removed L4: 5.6n, symbol Device:L
- removed Q1: 2N7002, Package_TO_SOT_SMD:SOT-23, symbol Transistor_FET:2N7002
- removed R1, R17, R2: 470, symbol Device:R
- removed R10, R14: 1M, symbol Device:R
- removed R11: 10K, symbol Device:R
- removed R12, R13, R9: 1k5, symbol Device:R
- removed R15, R19, R8: 10k, symbol Device:R
- removed R16: 4K7, symbol Device:R
- removed R18, R24, R26: 22k, symbol Device:R
- removed R20: 47k, symbol Device:R
- removed R21, R22: 100k, symbol Device:R
- removed R23, R25: 33k, symbol Device:R
- removed R3, R4, R5, R6: 4k7, symbol Device:R
- removed R7: 1k, symbol Device:R
- removed SW1, SW2: SW_SPDT, symbol Switch:SW_SPDT
- removed U1: STM32F405RGT6, Package_QFP:LQFP-64_10x10mm_P0.5mm, symbol MCU_ST_STM32F4:STM32F405RGTx
- removed U2: LM2596S-5, Package_TO_SOT_SMD:TO-263-5_TabPin3, symbol Regulator_Switching:LM2596S-5
- removed U3: AMS1117-3.3, Package_TO_SOT_SMD:SOT-223-3_TabPin2, symbol Regulator_Linear:AMS1117-3.3
- removed U4: MPU-6050, Sensor_Motion:InvenSense_QFN-24_4x4mm_P0.5mm, symbol Sensor_Motion:MPU-6050
- removed U5: HMC5883L, HMC5883L:HMC5883L, symbol HMC5883L:HMC5883L
- removed U6: SUP90P06-09L-E3, SUP90P06_09L_E3:TO-220AB_VIS, symbol SUP90P06_09L_E3:SUP90P06-09L-E3
- removed U7: nRF8001, Package_DFN_QFN:QFN-32-1EP_5x5mm_P0.5mm_EP3.45x3.45mm, symbol RF_Bluetooth:nRF8001
- removed U8: CH224K, Package_SO:SSOP-10-1EP_3.9x4.9mm_P1mm_EP2.1x3.3mm, symbol Interface_USB:CH224K
- removed Y1, Y4: 16MHz, symbol Device:Crystal_GND24
- removed Y3: 32.768kHz, symbol Device:Crystal_GND24
Connections:
- no-connect marks 40 -> 1
Other:
- added sheet BATTERY (battery.kicad_sch)
- added sheet COMMS (communication.kicad_sch)
- added sheet MICROCONTROLLER (mcu.kicad_sch)
- added sheet POWER SUPPLY (power_supply.kicad_sch)
- added sheet SENSORS (sensors.kicad_sch)
- note removed: "3.3V"
- note removed: "5V"
- note removed: "ANALOG FILTER"
- note removed: "BATTERY SENSOR"
- note removed: "BLUETHOOT LOW ENERGY"
- note removed: "COMPASS"
- note removed: "DECOUPLING CAPS"
- note removed: "EXTERNAL CLOCK"
- note removed: "I2C"
- note removed: "INERTIAL MEASUREMENT UNIT"
- note removed: "MICRO-SD"
- note removed: "MICROCONTROLLER"
- note removed: "ON/OFF SWITCH"
- note removed: "POWER SUPPLY"
- note removed: "PROGRAMMING BOOT"
- note removed: "SERIAL WIRE DEBUG"
- note removed: "SPI"
- note removed: "USB-C PROGRAMMING & CHARGER"
- moved on the sheet: H1, H2, H3, H4
